File: Hardware/12V_source.kicad_sch (KiCad schematic)
At the start: 4 parts, among them Q1601 NMOS

Commit message: inital schematic
Parts:
- removed D1601: D_Zener, symbol Device:D_Zener
- removed Q1601: NMOS, symbol Simulation_SPICE:NMOS
- added C1601, C1602: 4.7u 400V, symbol Device:C
- added C1603: 100n, symbol Device:C
- added C1604: 10u 25V, symbol Device:C
- added C1605: 100u 16V, symbol Device:C
- added D1601: 1N4007, symbol Device:D
- added D1602: UF4007, symbol Device:D
- added D1603: 1N4005GP, symbol Device:D
- added L1601: 1m, symbol Device:L
- added L1602: 1mH 280mA, symbol Device:L
- added R1603: 26.7k, PCM_JLCPCB:R_0402, symbol Device:R
- added R1604: 11.8k, PCM_JLCPCB:R_0402, symbol Device:R
- added R1605: 3.3k, PCM_JLCPCB:R_0402, symbol Device:R
- added U1601: LNK3204D-TL, lcsc_footprints:C567600_SO-8C_7P-L4_9-W3_9-P1_27-LS6_0-BL-PE3, symbol lcsc_imported:LNK3204D-TL
- R1601: value R -> 8R2 2W; footprint lcsc_footprints:C567600_SO-8C_7P-L4_9-W3_9-P1_27-LS6_0-BL-PE3 -> PCM_JLCPCB:R_0402
- R1602: value R -> 2.49k; footprint lcsc_footprints:C567600_SO-8C_7P-L4_9-W3_9-P1_27-LS6_0-BL-PE3 -> PCM_JLCPCB:R_0402
Connections:
- net +12V: now also C1605.1, D1603.2 (A), L1602.2, R1605.1; no longer R1602.1
- net GND: now also C1601.2, C1602.2, C1605.2, D1602.2 (A), R1605.2; no longer R1602.2
- net at R1601.2: now also D1601.2 (A)
- new net: C1601.1, D1601.1 (K), L1601.1
- new net: C1602.1, L1601.2, U1601.4 (D)
- new net: C1604.1, D1603.1 (K), R1603.2, R1604.2
- new net: R1602.1, R1604.1, U1601.2 (FB)
- new net: C1603.2, C1604.2, D1602.1 (K), L1602.1, R1602.2, U1601.5 (S), U1601.6 (S), U1601.7 (S), U1601.8 (S)
- new net: C1603.1, R1603.1, U1601.1 (BP/M)
Other:
- note added: "CHECK THIS"
- note added: "Like, This is for 230VAC and not 48VDC. Check this"
- note removed: "This boy gets hot"
