File: Hardware/Bus_switch.kicad_sch (KiCad schematic)
At the start: 15 parts, among them J301 Conn_01x04_Pin, U301 SN74CB3Q3384APW

Commit message: working commit
Parts:
- removed R310: 10kΩ, PCM_JLCPCB:R_0603, symbol PCM_JLCPCB-Resistors:0603,10kΩ
- removed U301: SN74CB3Q3384APW, Package_SO:TSSOP-24_4.4x7.8mm_P0.65mm, symbol 74xx:SN74CB3Q3384APW
- added R312: 10kΩ, PCM_JLCPCB:R_0603, symbol PCM_JLCPCB-Resistors:0603,10kΩ
- added U302: SN74CB3Q3245PWR, lcsc_footprints:C470961_TSSOP-20_L6_5-W4_4-P0_65-LS6_4-BL, symbol lcsc_imported:SN74CB3Q3245PWR
Connections:
- net +3V3: now also R312.1, U302.20 (VCC)
- net Chainbus.CS: now also U302.13 (B6)
- net Chainbus.MISO: now also U302.16 (B3)
- net Chainbus.MOSI: now also U302.15 (B4)
- net Chainbus.RX: now also U302.18 (B1)
- net Chainbus.SCK: now also U302.14 (B5)
- net Chainbus.SCL: now also U302.11 (B8)
- net Chainbus.SDA: now also U302.12 (B7)
- net Chainbus.TX: now also U302.17 (B2)
- net Chainbus_In.CS: now also U302.7 (A6)
- net Chainbus_In.MISO: now also U302.4 (A3)
- net Chainbus_In.MOSI: now also U302.5 (A4)
- net Chainbus_In.RX: now also U302.2 (A1)
- net Chainbus_In.SCK: now also U302.6 (A5)
- net Chainbus_In.SCL: now also U302.9 (A8)
- net Chainbus_In.SDA: now also U302.8 (A7)
- net Chainbus_In.TX: now also U302.3 (A2)
- net GND: now also U302.10 (GND)
- net SEL1: now also R312.2, U302.19 (OE#)
- no-connect marks 4 -> 1
Other:
- title: MMS3 Hat template small (Change Me) -> MMS3_hat_motor_high_power
- moved on the sheet: C301

Commit message: inital schematic
Parts:
- removed J301: Conn_01x04_Pin, Connector_PinHeader_2.54mm:PinHeader_1x04_P2.54mm_Vertical, symbol Connector:Conn_01x04_Pin
- removed R305, R306: 10kΩ, PCM_JLCPCB:R_0603, symbol PCM_JLCPCB-Resistors:0603,10kΩ
Connections:
- net Chainbus.RX: no longer names the net of U302.18 (B1)
- net Chainbus.TX: no longer names the net of U302.17 (B2)
- net Chainbus_In.RX: no longer names the net of U302.2 (A1)
- net Chainbus_In.TX: no longer names the net of U302.3 (A2)
- no-connect marks 1 -> 5
Other:
- note removed: "I2C Bus Connection"
- moved on the sheet: D301, R311
