File: Hardware/CH32V305RBT6.kicad_sch (KiCad schematic)
At the start: 32 parts, among them J1101 WCH Link, U1101 CH32V305RBT6, X1101 X322525MOB4SI, X1102 Q13FC1350000400

Commit message: inital schematic
Connections:
- net +3.3V is gone; now on net +3V3: J1101.8 (Pin_8), R1104.1, R1105.1, S1101.1 (A), S1102.1 (A)
