File: Hardware/CH32V305RBT6_wrapper.kicad_sch (KiCad schematic)
At the start: 0 parts

Commit message: inital schematic
Other:
- note added: "CHECK IF TIM CHANNELS FOR MOTOR ARE GOOD (IF EACH ONE IS TIMxCHx + TIMxCHxN"
- note added: "LEFT User usable GPIO"
- note added: "USE TIM1 and TIM3"
- note removed: "USE TIM1 and TIM8"
- note removed: "User usable GPIO"
