File: Hardware/Encoder.kicad_sch (KiCad schematic)
At the start: 1 part, among them J1301 Conn_01x06

Commit message: inital schematic
Parts:
- added D1301: D_TVS, symbol Device:D_TVS
- added R1301: 100Ω, PCM_JLCPCB:R_0402, symbol PCM_JLCPCB-Resistors:0402,100Ω
