File: Hardware/IO.kicad_sch (KiCad schematic)
At the start: 12 parts, among them J1501 Conn_01x02, J1502 Conn_01x02

Commit message: inital schematic
Parts:
- added D1505: D_TVS, symbol Device:D_TVS
- added R1507: 100Ω, PCM_JLCPCB:R_0402, symbol PCM_JLCPCB-Resistors:0402,100Ω
