File: Hardware/MMS3_hat_motor_high_power.kicad_pcb (KiCad board)
At the start: 2 copper layers, 100 x 50 mm, 132 parts, among them CN401 XT60PW-M, J1101 WCH Link, J1301 Conn_01x06, J201 Chainbus in, J202 Chainbus Out, J301 Conn_01x04_Pin, Q1001 XRS80N12F, Q1002 XRS80N12F, Q704 XRS80N12F, Q705 XRS80N12F, Q801 XRS80N12F, Q802 XRS80N12F, Q901 XRS80N12F, Q902 XRS80N12F, U1001 UCC27302ADRCR, U1002 INA181A2IDBVR(LX), U101 AMS1117, U1101 CH32V305RBT6, U302 SN74CB3Q3245PWR, U401 XT60PW-F_C428722, U501 M24C64, U601 AMS1117, U701 UCC27302ADRCR, U702 INA181A2IDBVR(LX), U801 UCC27302ADRCR, U802 INA181A2IDBVR(LX), U901 UCC27302ADRCR, U902 INA181A2IDBVR(LX), X1101 X322525MOB4SI, X1102 Q13FC1350000400

Commit message: inital schematic
Parts:
- removed C602, C603: 10uF, PCM_JLCPCB:C_0603
- removed J301: Conn_01x04_Pin, Connector_PinHeader_2.54mm:PinHeader_1x04_P2.54mm_Vertical
- removed R305, R306: 10kΩ, PCM_JLCPCB:R_0603
- added D1001: D_TVS, PCM_JLCPCB:R_0402, F.Cu at (211.4, 124.3)
- added D1501: Red, PCM_JLCPCB:D_0603, F.Cu at (257.7, 112.2)
- added D1502: Red, PCM_JLCPCB:D_0603, F.Cu at (257.7, 114.8)
- added D1503: Red, PCM_JLCPCB:D_0603, F.Cu at (257.7, 117.4)
- added D1504: Red, PCM_JLCPCB:D_0603, F.Cu at (257.7, 120.0)
- added D601: Red, PCM_JLCPCB:D_0603, F.Cu at (254.8, 94.2)
- added D607: Red, PCM_JLCPCB:D_0603, F.Cu at (254.8, 99.4)
- added D701: D_TVS, PCM_JLCPCB:R_0402, F.Cu at (236.0, 97.5)
- added D801: D_TVS, PCM_JLCPCB:R_0402, F.Cu at (236.0, 115.5)
- added D901: D_TVS, PCM_JLCPCB:R_0402, F.Cu at (236.0, 133.5)
- added J1501: Conn_01x02, Connector_JST:JST_XH_S2B-XH-A-1_1x02_P2.50mm_Horizontal, F.Cu at (157.7, 129.2)
- added J1502: Conn_01x02, Connector_JST:JST_XH_S2B-XH-A-1_1x02_P2.50mm_Horizontal, F.Cu at (167.1, 129.2)
- added R1501: 1kΩ, PCM_JLCPCB:R_0402, F.Cu at (254.2, 111.8)
- added R1502: 1kΩ, PCM_JLCPCB:R_0402, F.Cu at (254.2, 113.7)
- added R1503: 1kΩ, PCM_JLCPCB:R_0402, F.Cu at (254.2, 115.5)
- added R1504: 1kΩ, PCM_JLCPCB:R_0402, F.Cu at (254.2, 117.4)
- added R1505: 10kΩ, PCM_JLCPCB:R_0402, F.Cu at (254.2, 119.2)
- added R1506: 10kΩ, PCM_JLCPCB:R_0402, F.Cu at (254.2, 121.1)
- added R603: 1kΩ, PCM_JLCPCB:R_0402, F.Cu at (258.3, 95.7)
- added R604: 220kΩ, PCM_JLCPCB:R_0603, F.Cu at (258.7, 101.8)
- added R605: 12kΩ, PCM_JLCPCB:R_0402, F.Cu at (258.3, 97.5)
- added U1601: LNK3204D-TL, lcsc_footprints:C567600_SO-8C_7P-L4_9-W3_9-P1_27-LS6_0-BL-PE3, F.Cu at (213.7, 141.7)
- added U602: XT60PW-F_C428722, lcsc_footprints:C428722_TH_2P-XT60PW-F, F.Cu at (128.9, 130.8)
- added U603: MR30PW-F20.G.Y, lcsc_footprints:C19268035_CONN-TH_MR30PW-F, F.Cu at (128.9, 133.5)
- U601: value AMS1117 -> XT60PW-F_C428722; footprint PCM_JLCPCB:SOT-223_L6.5-W3.5-P2.30-LS7.0-BR -> lcsc_footprints:C428722_TH_2P-XT60PW-F
- moved U601 97.7 mm to (145.7, 130.8), turned to 180 degrees
- moved J1301 62.0 mm to (156.8, 134.3)
- moved S1101 58.7 mm to (176.3, 113.4)
- moved S1102 58.7 mm to (176.3, 117.8)
- moved S1103 58.7 mm to (176.3, 122.3)
- moved R602 48.5 mm to (258.3, 93.8)
- moved D603 43.8 mm to (254.8, 96.8)
- moved C1001 41.3 mm to (220.0, 134.1)
- moved U1002 41.3 mm to (220.3, 130.4)
- moved R601 40.9 mm to (258.7, 99.6)
- moved R1001 39.7 mm to (211.4, 126.1)
- moved R1003 39.7 mm to (211.4, 128.0)
- moved R1004 39.7 mm to (211.4, 129.8)
- moved R1006 39.7 mm to (211.4, 131.7)
- moved R1007 39.7 mm to (211.4, 133.5)
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Connections:
- D603 pad 1: unconnected-(D603-Pad1) -> GND
- D603 pad 2: unconnected-(D603-Pad2) -> Net-(D603-Pad2)
- J1101 pad 8: +3.3V -> +3V3
- J201 pad 30: /Bus_switch/Chainbus_In.TX -> /Interboard_connector/Chainbus.TX
- J201 pad 32: /Bus_switch/Chainbus_In.RX -> /Interboard_connector/Chainbus.RX
- J202 pad 30: /Bus_switch/Chainbus_In.TX -> /Interboard_connector/Chainbus.TX
- J202 pad 32: /Bus_switch/Chainbus_In.RX -> /Interboard_connector/Chainbus.RX
- R1104 pad 1: +3.3V -> +3V3
- R1105 pad 1: +3.3V -> +3V3
- R1401 pad 2: /User Area/CH32V305RBT6/TempADC -> /User Area/CH32V305RBT6/GPIOA3
- R601 pad 2: /User Area/Ubus -> /User Area/CH32V305RBT6/GPIOB0
- R602 pad 1: /User Area/Ubus -> /User Area/CH32V305RBT6/GPIOB0
- S1101 pad 1: +3.3V -> +3V3
- S1102 pad 1: +3.3V -> +3V3
- U1001 pad 6: /User Area/Mosfet_EN -> /User Area/CH32V305RBT6/GPIOB12
- U1101 pad 10: /User Area/CH32V305RBT6/GPIOC2 -> /User Area/ADC2
- U1101 pad 11: /User Area/CH32V305RBT6/GPIOC3 -> /User Area/ADC3
- U1101 pad 15: /User Area/CH32V305RBT6/GPIOA1 -> /User Area/ADC6
- U1101 pad 16: /User Area/CH32V305RBT6/GPIOA2 -> /User Area/ADC7
- U1101 pad 24: /User Area/CH32V305RBT6/GPIOC4 -> /User Area/ADC4
- U1101 pad 25: /User Area/CH32V305RBT6/GPIOC5 -> /User Area/ADC5
- U1101 pad 8: /User Area/CH32V305RBT6/GPIOC0 -> /User Area/ADC0
- U1101 pad 9: /User Area/CH32V305RBT6/GPIOC1 -> /User Area/ADC1
- U302 pad 17: /Bus_switch/Chainbus.TX -> unconnected-(U302-B2-Pad17)
- U302 pad 18: /Bus_switch/Chainbus.RX -> unconnected-(U302-B1-Pad18)
- U302 pad 2: /Bus_switch/Chainbus_In.RX -> unconnected-(U302-A1-Pad2)
- U302 pad 3: /Bus_switch/Chainbus_In.TX -> unconnected-(U302-A2-Pad3)
- U601 pad 1: GND -> unconnected-(U601-Pad1)
- U601 pad 2: Net-(D601-A) -> unconnected-(U601-Pad2)
- U601 pad 3: +12V -> /User Area/Half H bridge2/HS
- U601 pad 4: Net-(D601-A) -> /User Area/Half H bridge3/HS
- U701 pad 6: /User Area/Mosfet_EN -> /User Area/CH32V305RBT6/GPIOB12
- U801 pad 6: /User Area/Mosfet_EN -> /User Area/CH32V305RBT6/GPIOB12
- U901 pad 6: /User Area/Mosfet_EN -> /User Area/CH32V305RBT6/GPIOB12
