File: Hardware/MMS3_hat_motor_high_power.kicad_sch (KiCad schematic)
At the start: 9 parts, among them U101 AMS1117

Commit message: inital schematic
Other:
- note removed: "-> when using >48V unsolder D401"
- note removed: "Up to 100V 10A"
- note removed: "Up to 48V"
Changed lines of the file:
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@@
-		)
-	)
-	(text "Up to 100V 10A"
-		(exclude_from_sim no)
-		(at 114.554 127 0)
-		(effects
-			(font
-				(size 1.27 1.27)
-			)
 		)
 	)
@@
 			)
 		)
-	)
-	(text "Up to 48V"
-		(exclude_from_sim no)
-		(at 109.728 140.462 0)
-		(effects
-			(font
-				(size 1.27 1.27)
-			)
-		)
-	)
-	(text "-> when using >48V unsolder D401"
-		(exclude_from_sim no)
-		(at 116.332 129.286 0)
-		(effects
-			(font
-				(size 1.27 1.27)
-			)
-		)
