File: Hardware/Power_Connector.kicad_sch (KiCad schematic)
At the start: 3 parts, among them J401 AMASS XT60 Male, J402 AMASS XT60 Female

Commit message: working commit
Parts:
- removed J401: AMASS XT60 Male, XT60:AMASS_XT60PW-M_1x02_P7.20mm_Horizontal, symbol Connector_Generic:Conn_01x02
- removed J402: AMASS XT60 Female, XT60:AMASS_XT60PW-F_1x02_P7.20mm_Horizontal, symbol Connector_Generic:Conn_01x02
- added CN401: XT60PW-M, lcsc_footprints:C98732_CONN-TH_XT60PW-M, symbol lcsc_imported:XT60PW-M
- added U401: XT60PW-F_C428722, lcsc_footprints:C428722_TH_2P-XT60PW-F, symbol lcsc_imported:XT60PW-F_C428722
Connections:
- net GND: now also CN401.1 (-), U401.4 (-)
- net VIN_BRD: now also CN401.2 (+), U401.3 (+)
- no-connect marks 0 -> 4
Other:
- title: MMS3 Hat template small (Change Me) -> MMS3_hat_motor_high_power

Commit message: inital schematic
Parts:
- added D402: Red, PCM_JLCPCB:D_0603, symbol PCM_JLCPCB-Diodes:LED,0603,Red
- added R401: 27kΩ, PCM_JLCPCB:R_0603, symbol PCM_JLCPCB-Resistors:0603,27kΩ
Connections:
- net GND: now also D402.1
- net VIN_BRD: now also R401.1
- new net: D402.2, R401.2
Other:
- moved on the sheet: D401
