File: Hardware/UCC27302ADRCR_Half_H_Bridge.kicad_sch (KiCad schematic)
At the start: 17 parts, among them Q704 XRS80N12F, Q705 XRS80N12F, U701 UCC27302ADRCR, U702 INA181A2IDBVR(LX)

Commit message: inital schematic
Parts:
- removed R703: 220kΩ, PCM_JLCPCB:R_0603, symbol PCM_JLCPCB-Resistors:0603,220kΩ
- removed R704: 6.8kΩ, PCM_JLCPCB:R_0402, symbol PCM_JLCPCB-Resistors:0402,6.8kΩ
- added C705: 100nF, PCM_JLCPCB:C_0805, symbol PCM_JLCPCB-Capacitors:0805,100nF
- added C706: 1uF, PCM_JLCPCB:C_0805, symbol Device:C
- added R703: 47kΩ, PCM_JLCPCB:R_0402, symbol PCM_JLCPCB-Resistors:0402,47kΩ
- added R704: 3.3kΩ, PCM_JLCPCB:R_0402, symbol PCM_JLCPCB-Resistors:0402,3.3kΩ
- added R708, R709: 10kΩ, PCM_JLCPCB:R_0402, symbol PCM_JLCPCB-Resistors:0402,10kΩ
- D701: footprint PCM_JLCPCB:R_0402 -> (none)
- R705: value SHUNT 5mohm -> SHUNT 2.5mohm
Connections:
- net GND: now also C705.2, C706.2, R704.2
- net OUT: now also R703.1, R708.2
- net Shunt+: now also R709.2
- net VIN: now also C705.1, C706.1
- net Vmes: now also R703.2, R704.1
- net at Q705.4 (G), R702.2: now also R709.1
- net at Q704.4 (G), R701.2: now also R708.1
Other:
- note added: "Layout Shunt- as a trace, don't use global GND"
