File: Hardware/User_area.kicad_sch (KiCad schematic)
At the start: 13 parts, among them J601 Conn_01x02, J602 Conn_01x03, J603 Conn_01x02

Commit message: inital schematic
Parts:
- removed J601, J603: Conn_01x02, PCM_JLCPCB:R_0402, symbol Connector_Generic:Conn_01x02
- removed J602: Conn_01x03, PCM_JLCPCB:R_0402, symbol Connector_Generic:Conn_01x03
- removed R601, R604: 220kΩ, PCM_JLCPCB:R_0603, symbol PCM_JLCPCB-Resistors:0603,220kΩ
- removed R602: 6.8kΩ, PCM_JLCPCB:R_0402, symbol PCM_JLCPCB-Resistors:0402,6.8kΩ
- added R601: 3.3kΩ, PCM_JLCPCB:R_0402, symbol PCM_JLCPCB-Resistors:0402,3.3kΩ
- added R602: 10kΩ, PCM_JLCPCB:R_0402, symbol PCM_JLCPCB-Resistors:0402,10kΩ
- added R604, R606: 47kΩ, PCM_JLCPCB:R_0402, symbol PCM_JLCPCB-Resistors:0402,47kΩ
- added U601, U602: XT60PW-F_C428722, lcsc_footprints:C428722_TH_2P-XT60PW-F, symbol lcsc_imported:XT60PW-F_C428722
- added U603: MR30PW-F20.G.Y, lcsc_footprints:C19268035_CONN-TH_MR30PW-F, symbol lcsc_imported:MR30PW-F20_G_Y
Connections:
- net GND: now also R601.2, R602.2
- net Half H bridge/OUT: now also U602.3 (+), U603.1
- net Half H bridge1/OUT: now also U602.4 (-), U603.2
- net Half H bridge2/OUT: now also U601.3 (+), U603.3
- net Half H bridge3/OUT: now also U601.4 (-)
- net Mosfet_EN: now also R602.1
- net Ubus: now also R601.1, R604.2
- net VIN: now also R604.1, R606.1
- net at D607.2: now also R606.2
- no-connect marks 2 -> 8
Other:
- sheet CH32V305RBT6 ports: added {Mosfet_EN}, {Ubus}; removed Mosfet_EN, UbusADC
- note added: "ADD BULK CAPS TO EACH LINE"
- note added: "ADD R IN SERIES TO LOGIC LINES SO YOU WONT FRY IT WHEN SHORTING + ADD TVS DIODES"
- note added: "ADD SOME KIND OF THING TO SHORT FOR LOW VOLTAGE VBUS"
- note added: "C_POLAR is bulk"
